File: eclipse_sao_v1/eclipse_sao_v1.kicad_sch (KiCad schematic)
At the start: 11 parts, among them J101 SAO 1.69bis

Commit message: Schematic
Other:
- note added: "I2C and GPIO Termination"
- note added: "SAO Connector"
- company: (none) -> AB4EN - Sky Iron Studio
- title: (none) -> Eclipse SAO
- moved on the sheet: D105, J101, R105
